Commit message: Actualizado URDF de 4 ruedas con colisiones e inercias

File: src/robot_4_ruedas_description/urdf/robot_4_ruedas.urdf (robot description, URDF)
Before this commit: robot carreta_robot, 5 links, 4 joints
Links:
- added link base_footprint
Joints:
- added joint base_footprint_joint: type fixed, parent base_footprint, child base_link, origin xyz=0 0 0 rpy=0 0 0
- joint front_left_wheel_joint: limit lower=-6.28 upper=6.28 effort=1 velocity=1 -> lower=-3.14 upper=3.14 effort=100 velocity=10; origin xyz=0.17 0.20 0.1 rpy=0 0 0 -> xyz=0.2 0.225 0.1 rpy=0 0 0
- joint front_right_wheel_joint: limit lower=-6.28 upper=6.28 effort=1 velocity=1 -> lower=-3.14 upper=3.14 effort=100 velocity=10; origin xyz=0.17 -0.20 0.1 rpy=0 0 0 -> xyz=0.2 -0.225 0.1 rpy=0 0 0
- joint left_wheel_joint: limit lower=-6.28 upper=6.28 effort=1 velocity=1 -> lower=-3.14 upper=3.14 effort=100 velocity=10; origin xyz=-0.17 0.20 0.1 rpy=0 0 0 -> xyz=-0.2 0.225 0.1 rpy=0 0 0
- joint right_wheel_joint: limit lower=-6.28 upper=6.28 effort=1 velocity=1 -> lower=-3.14 upper=3.14 effort=100 velocity=10; origin xyz=-0.17 -0.20 0.1 rpy=0 0 0 -> xyz=-0.2 -0.225 0.1 rpy=0 0 0
